File: STS1_connector.sch (KiCad schematic (older format))
At the start: 2 parts

Commit message: Made some changes to file structure, schematic and PCB - Unzipped the zip - KiCAD libraries should no be imported with relative pathes. - Copper layer IN1 is now connected to GND - Copper layer IN2 is now connected to output voltage. - Connected VBUS and GND of the CSBI to the output voltage and GND. - Modified some vias.
Connections:
- wire segments 66 -> 77
- no-connect marks 8 -> 0
Changed lines of the file:
@@
 	3450 2850 3950 2850
-Wire Wire Line
-	3450 2950 3950 2950
 Wire Wire Line
 	3450 3050 3950 3050
@@
 Wire Wire Line
 	6500 3900 7000 3900
-Wire Wire Line
-	6500 4000 7000 4000
-Wire Wire Line
-	6500 4100 7000 4100
 $Comp
 L power:GND #PWR042
@@
 Connection ~ 3450 1850
 $Comp
-L power:VBUS #PWR045
-U 1 1 617AD547
-P 3450 1950
-F 0 "#PWR045" H 3450 1800 50  0001 C CNN
-F 1 "VBUS" V 3465 2077 50  0000 L CNN
-F 2 "" H 3450 1950 50  0001 C CNN
-F 3 "" H 3450 1950 50  0001 C CNN
-	1    3450 1950
-	0    -1   -1   0
-$EndComp
-Connection ~ 3450 1950
-$Comp
-L power:VBUS #PWR046
-U 1 1 617ADEFD
-P 3450 2050
-F 0 "#PWR046" H 3450 1900 50  0001 C CNN
-F 1 "VBUS" V 3465 2177 50  0000 L CNN
-F 2 "" H 3450 2050 50  0001 C CNN
-F 3 "" H 3450 2050 50  0001 C CNN
-	1    3450 2050
-	0    -1   -1   0
-$EndComp
-Connection ~ 3450 2050
-$Comp
 L power:GND #PWR047
 U 1 1 617AE72F
@@
 L power:GND #PWR050
 U 1 1 617B045A
-P 3450 2950
-F 0 "#PWR050" H 3450 2700 50  0001 C CNN
-F 1 "GND" V 3455 2822 50  0000 R CNN
-F 2 "" H 3450 2950 50  0001 C CNN
-F 3 "" H 3450 2950 50  0001 C CNN
-	1    3450 2950
-	0    1    1    0
-$EndComp
-Connection ~ 3450 2950
+P 3350 2950
+F 0 "#PWR050" H 3350 2700 50  0001 C CNN
+F 1 "GND" V 3355 2822 50  0000 R CNN
+F 2 "" H 3350 2950 50  0001 C CNN
+F 3 "" H 3350 2950 50  0001 C CNN
+	1    3350 2950
+	0    1    1    0
+$EndComp
 Wire Wire Line
 	3450 3050 2850 3050
@@
 EDU_SPI_6
 $Comp
-L power:GND #PWR052
-U 1 1 617B97C4
-P 3450 3650
-F 0 "#PWR052" H 3450 3400 50  0001 C CNN
-F 1 "GND" V 3455 3522 50  0000 R CNN
-F 2 "" H 3450 3650 50  0001 C CNN
-F 3 "" H 3450 3650 50  0001 C CNN
-	1    3450 3650
-	0    1    1    0
-$EndComp
-Connection ~ 3450 3650
-$Comp
 L power:GND #PWR057
 U 1 1 617B9D0C
@@
 L power:GND #PWR058
 U 1 1 617C4645
-P 6500 4100
-F 0 "#PWR058" H 6500 3850 50  0001 C CNN
-F 1 "GND" V 6505 3972 50  0000 R CNN
-F 2 "" H 6500 4100 50  0001 C CNN
-F 3 "" H 6500 4100 50  0001 C CNN
-	1    6500 4100
-	0    1    1    0
-$EndComp
-Connection ~ 6500 4100
+P 6350 4100
+F 0 "#PWR058" H 6350 3850 50  0001 C CNN
+F 1 "GND" V 6355 3972 50  0000 R CNN
+F 2 "" H 6350 4100 50  0001 C CNN
+F 3 "" H 6350 4100 50  0001 C CNN
+	1    6350 4100
+	0    1    1    0
+$EndComp
 $Comp
 L power:GND #PWR056
 U 1 1 617C4E49
-P 6500 4000
-F 0 "#PWR056" H 6500 3750 50  0001 C CNN
-F 1 "GND" V 6505 3872 50  0000 R CNN
-F 2 "" H 6500 4000 50  0001 C CNN
-F 3 "" H 6500 4000 50  0001 C CNN
-	1    6500 4000
-	0    1    1    0
-$EndComp
-Connection ~ 6500 4000
+P 6350 4000
+F 0 "#PWR056" H 6350 3750 50  0001 C CNN
+F 1 "GND" V 6355 3872 50  0000 R CNN
+F 2 "" H 6350 4000 50  0001 C CNN
+F 3 "" H 6350 4000 50  0001 C CNN
+	1    6350 4000
+	0    1    1    0
+$EndComp
 Wire Wire Line
 	6500 3600 6000 3600
@@
 $EndComp
 Connection ~ 6500 3700
-$Comp
-L power:VBUS #PWR054
-U 1 1 6180C534
-P 6500 3800
-F 0 "#PWR054" H 6500 3650 50  0001 C CNN
-F 1 "VBUS" V 6515 3927 50  0000 L CNN
-F 2 "" H 6500 3800 50  0001 C CNN
-F 3 "" H 6500 3800 50  0001 C CNN
-	1    6500 3800
-	0    -1   -1   0
-$EndComp
-Connection ~ 6500 3800
-$Comp
-L power:VBUS #PWR055
-U 1 1 6180CCF4
-P 6500 3900
-F 0 "#PWR055" H 6500 3750 50  0001 C CNN
-F 1 "VBUS" V 6515 4027 50  0000 L CNN
-F 2 "" H 6500 3900 50  0001 C CNN
-F 3 "" H 6500 3900 50  0001 C CNN
-	1    6500 3900
-	0    -1   -1   0
-$EndComp
-Connection ~ 6500 3900
-NoConn ~ 3450 2250
-NoConn ~ 3450 3750
-NoConn ~ 3450 3850
-NoConn ~ 3450 3950
-NoConn ~ 6500 1900
-NoConn ~ 6500 2000
-NoConn ~ 6500 2100
-NoConn ~ 6500 2200
 Text Notes 4650 2200 0    50   ~ 0
 For UART the numbering is as follows\n1: TX\n2: RX\n
+Text HLabel 2800 1950 0    50   Input ~ 0
+VBUS
+Wire Wire Line
+	2800 1950 3350 1950
+Connection ~ 3450 1950
+Wire Wire Line
+	3350 1950 3350 2050
+Wire Wire Line
+	3350 2050 3450 2050
+Connection ~ 3350 1950
+Wire Wire Line
+	3350 1950 3450 1950
+Connection ~ 3450 2050
+Text HLabel 5900 3800 0    50   Input ~ 0
+VBUS
+Connection ~ 6500 3800
+Wire Wire Line
+	6400 3800 6400 3900
+Wire Wire Line
+	6400 3900 6500 3900
+Wire Wire Line
+	5900 3800 6400 3800
+Connection ~ 6400 3800
+Wire Wire Line
+	6400 3800 6500 3800
+Connection ~ 6500 3900
+Wire Wire Line
+	3950 2950 3450 2950
+Connection ~ 3450 2950
+Wire Wire Line
+	3450 2950 3350 2950
+Wire Wire Line
+	7000 4000 6500 4000
+Connection ~ 6500 4000
+Wire Wire Line
+	6500 4000 6350 4000
+Wire Wire Line
+	7000 4100 6500 4100
 Wire Bus Line
 	5900 3200 5900 3700
 Wire Bus Line
 	2750 3150 2750 3900
+Connection ~ 6500 4100
+Wire Wire Line
+	6500 4100 6350 4100
+$Comp
+L power:GND #PWR0106
+U 1 1 61C414EB
+P 3450 3650
+F 0 "#PWR0106" H 3450 3400 50  0001 C CNN
+F 1 "GND" V 3455 3522 50  0000 R CNN
+F 2 "" H 3450 3650 50  0001 C CNN
+F 3 "" H 3450 3650 50  0001 C CNN
+	1    3450 3650
+	0    1    1    0
+$EndComp
+Connection ~ 3450 3650
 $EndSCHEMATC
