File: STS1_template.sch (KiCad schematic (older format))
At the start: 51 parts, among them J1 SCC_Eingang, J2 BCC_Ausgang, J3 Battery_Anschluss, J4 Screw_Terminal_01x02, U1 coordinate_system, U2 ltc4040eufd-trpbf, U3 SIS488DN-T1-GE3

Commit message: Made some changes to file structure, schematic and PCB - Unzipped the zip - KiCAD libraries should no be imported with relative pathes. - Copper layer IN1 is now connected to GND - Copper layer IN2 is now connected to output voltage. - Connected VBUS and GND of the CSBI to the output voltage and GND. - Modified some vias.
Parts:
- MOSFET1: symbol SIR424DP-T1-GE3:SIR424DP-T1-GE3 -> 2021-12-02_18-12-51:SIR424DP-T1-GE3
- U2: symbol LTC4040_neu_2:ltc4040eufd-trpbf -> 2021-11-29_12-35-30:ltc4040eufd-trpbf
- U3: symbol SiS488DN:SIS488DN-T1-GE3 -> 2021-12-02_20-00-05:SIS488DN-T1-GE3
Connections:
- wire segments 168 -> 166
- no-connect marks 0 -> 1
